File: Hardware/LM3671_Buck_Converter_Module/LM3671_Buck_Converter_Module.kicad_pcb (KiCad board)
At the start: 2 copper layers, 17.9 x 12 mm, 8 parts, among them U1 LM3671MFX-3.3_NOPB

Commit message: updated rxver and txver hardware
Parts:
- removed J2, J3: ~, Connector_PinHeader_2.54mm:PinHeader_1x01_P2.54mm_Vertical
- J1: value ~ -> Conn_01x03_Pin; footprint Connector_PinHeader_2.54mm:PinHeader_1x01_P2.54mm_Vertical -> Connector_PinHeader_2.54mm:PinHeader_1x03_P2.54mm_Vertical; moved to F.Cu
- moved J1 6.41 mm to (103.9, 82.2), turned to -90 degrees
Routing:
- net Net-(U1-EN): track 3.85 -> 1.74 mm
- net GND: vias 8 -> 4
Other:
- board size 17.9 x 12 mm -> 11.7 x 12 mm
