File: Hardware/MotoHud_Project/MotoHud_Project.kicad_pcb (KiCad board)
At the start: 2 copper layers, 31.8 x 74.7 mm, 9 parts, among them J1 I2C, J2 BAT CHARGER, J3 Conn_01x02_Pin, J4 BTN

Commit message: updated rxver and txver hardware
Parts:
- R1, R2: footprint Resistor_THT:R_Axial_DIN0207_L6.3mm_D2.5mm_P7.62mm_Horizontal -> Resistor_SMD:R_0603_1608Metric_Pad0.98x0.95mm_HandSolder; moved to B.Cu
- moved R1 5.87 mm to (105.1, 84.9)
- moved R2 0.81 mm to (105.1, 88.0)
- moved J1 0.30 mm to (92.2, 126.4)
Routing:
- net GND: track 0.16 -> 16.0 mm, vias 0 -> 4
- net VDD: track 105.2 -> 108.9 mm
- net VBAT: track 64.5 -> 60.9 mm
- net Net-(B1-PadPA0): track 5.56 -> 4.84 mm
- net SDA: track 31.1 -> 31.8 mm

Commit message: updated hardware
Parts:
- removed J1: I2C, Connector_PinHeader_2.54mm:PinHeader_1x04_P2.54mm_Vertical
- added R3: R_PUP, Resistor_THT:R_Axial_DIN0207_L6.3mm_D2.5mm_P10.16mm_Horizontal, F.Cu at (92.9, 97.8)
- added R4: R_PUP, Resistor_THT:R_Axial_DIN0207_L6.3mm_D2.5mm_P10.16mm_Horizontal, F.Cu at (92.9, 101.5)
- added U2: 3.5mm_AudioJack_PJ-320A, CUSTOM_MODULES:3.5mm_AudioJack_PJ-320A_NoGuide, F.Cu at (87.5, 117.2)
Routing:
- net SCL: track 36.4 -> 27.6 mm
- net GND: track 16.0 -> 24.7 mm, vias 4 -> 6
- net VDD: track 108.9 -> 114.6 mm
- net SDA: track 31.8 -> 30.8 mm
